File: VCF.kicad_sch (KiCad schematic)
At the start: 26 parts

Commit message: Replace schematic
Parts:
- removed R?: 1k, symbol Device:R_Small
- removed R?: 20k, symbol Device:R_Small
- removed R?: 100k, symbol Device:R_Small
- added C? (x4): 1uF, symbol Device:C_Small
- added C? (x4): 100nF, symbol Device:C_Small
- added J? (x4): PJ301M-12, symbol eurocad:PJ301M-12
- added R? (x8): 10k, symbol Device:R_Small
- added R?: 100k, symbol Device:R_Small
- added R?: 20k, symbol Device:R_Small
- added R? (x2): 15k, symbol Device:R_Small
- added R?: 30k, symbol Device:R_Small
- added RV?: R_Potentiometer, symbol Device:R_Potentiometer
- added U? (x5): TL084, symbol Amplifier_Operational:TL084
- C? (x2): value 68nF -> 10nF
- RV?: value R_Potentiometer -> 100k
Connections:
- net +12V: now also RV?.1, C?.1, C?.1, U?.4 (V+)
- net -12V: now also RV?.3, C?.2, C?.2, U?.11 (V-)
- net BIAS: now also R?.1, R?.1; no longer RV?.2, RV?.3, U?.5 (BIAS), U?.5 (BIAS)
- net GND: now also U?.3 (+), C?.1, C?.1, C?.2, C?.2, J?.2, J?.2, J?.2, J?.2, J?.3, J?.3, J?.3, J?.3, R?.2, R?.2, R?.2, R?.2, RV?.3
- net at C?.1, R?.2, U?.6: now also U?.10 (+); no longer U?.5 (+)
- net TP: now reaches U?.14
- net TP: now also R?.1, U?.12 (+), C?.1
- net BP: now reaches R?.1, R?.2
- net BP: now also U?.8, U?.9 (-), C?.1; no longer U?.6 (-), U?.7
- net at C?.1, R?.2, U?.6: now also U?.13 (-); no longer U?.10 (+)
- net at R?.1, R?.2: now also U?.5 (+); no longer U?.3 (+)
- net at R?.1, R?.2, R?.2: now also U?.6 (-); no longer U?.2 (-)
- net at R?.2: now also U?.1, R?.1
- net HP: now reaches R?.1, R?.1
- net HP: now also U?.7, C?.1; no longer U?.1
- new net: C?.2, U?.10 (+)
- new net: R?.1, R?.2, U?.6 (-)
- new net: R?.2, U?.5 (BIAS) (x2)
- new net: R?.1, RV?.2, U?.3 (+)
- new net: R?.2, RV?.2
- new net: C?.2, U?.5 (+)
- new net: R?.1, R?.2, U?.9 (-)
- new net: R?.1, R?.2, U?.12 (+)
- new net: C?.2, U?.13 (-)
- new net: R?.1, R?.2, U?.2 (-)
- new net: C?.2, R?.2
- new net: R?.1, R?.2
- new net AUDIO_IN: C?.1
- new net BP_OUT: J?.1, R?.1, U?.8
- new net Bias: U?.1, U?.2 (-)
- new net FREQ_CV_IN: J?.1, RV?.1
- new net HP_OUT: J?.1, R?.1, U?.14
- new net TP_OUT: J?.1, R?.1, U?.7
Other:
- added sheet Inputs & Outputs (in_out.kicad_sch)
- company: (none) -> Audioschaltungstechnik - BHT Berlin
- title: (none) -> Voltage Controlled State Variable Filter
- moved on the sheet: C?, R?, RV?, U?, U?A, U?B, U?C, U?D, U?E
