File: VCF.kicad_sch (KiCad schematic)
At the start: 53 parts, among them J1 CV_IN, J2 TP_OUT, J3 BP_OUT, J4 HP_OUT, U1 TL084, U2 TL084, U3 CA3080, U4 CA3080

Commit message: Add files via upload
First Layout Draft (Not Complete!) 
Current File: VCF. Only for measuring the layout
Parts:
- added H2: (no value), symbol Mechanical:MountingHole_Pad
- added J5: (no value), Connector_Audio:Jack_3.5mm_QingPu_WQP-PJ398SM_Vertical_CircularHoles, symbol Connector:AudioJack2_SwitchT
- added RV3, RV4: 100k, Potentiometer_THT:Potentiometer_Alpha_RD901F-40-00D_Single_Vertical_CircularHoles, symbol Device:R_Potentiometer
- U1, U2: value TL084 -> (none); footprint Package_DIP:DIP-14_W7.62mm_Socket -> (none)
- U1: renamed from U2; value TL084 -> (none); footprint Package_DIP:DIP-14_W7.62mm_Socket -> (none)
- U2: renamed from U1; value TL084 -> (none); footprint Package_DIP:DIP-14_W7.62mm_Socket -> (none)
- renumbered C13 to C12, C14 to C13, C3 to C14, C12 to C3
Connections:
- net BP: now also U2.1, U2.2 (-), RV4.1, RV4.2; no longer R14.1, U2.8, U2.9 (-)
- net BP_OUT: now also U1.7; no longer U1.8
- net Bias: now also U1.14; no longer U1.1
- net GND: now also U2.10 (+), H2.1, J5.S, J5.TN, RV3.3; no longer U2.3 (+)
- net HP: now also U2.14; no longer U2.7
- net HP_OUT: now also U1.8; no longer U1.14
- net TP: now also U2.5 (+), U2.7; no longer U2.12 (+), U2.14
- net TP_OUT: now also U1.1; no longer U1.7
- net at C3.2: now also U1.5 (+); no longer U1.10 (+)
- net at R2.2, R3.1: now also U1.2 (-); no longer U1.6 (-)
- net at C15.1, R16.2, U3.6: now also U2.3 (+); no longer U2.10 (+)
- net at R14.2, R8.1: now also U2.12 (+); no longer U2.5 (+)
- net at R20.2, R7.1, R9.2: now also U2.13 (-); no longer U2.6 (-)
- net at R27.2, R28.1: now also U1.13 (-); no longer U1.2 (-)
- net at C16.1, R26.2, U4.6: now also U2.6 (-); no longer U2.13 (-)
- net at R22.1, R23.1, R25.1: now also U1.12 (+); no longer U1.3 (+)
- net at C1.2: now also U1.3 (+); no longer U1.5 (+)
- net at R10.2, R11.1: now also U1.6 (-); no longer U1.9 (-)
- net at R4.2, R5.1: now also U1.10 (+); no longer U1.12 (+)
- net at C2.2: now also U1.9 (-); no longer U1.13 (-)
- net at R1.1, R6.2: now also U2.9 (-); no longer U2.2 (-)
- net at R6.1, R7.2: now also U2.8; no longer U2.1
- net AUDIO_IN: no longer names the net of C14.1
- net AUDIO_IN: now also RV3.2
- new net: R14.1, RV4.3
- new net AUDIO_IN_ATT: J5.T, RV3.1
Other:
- moved on the sheet: J1, J2, J3, J4

Commit message: Prototype #1
Layout and Schematics Done. 
Please ignore Silkscreen, SolderPaste and Courtyard warnings; won't be manufactured! 
Check M3 mounting hole size and position and the GND Vias!
Parts:
- H2: value (none) -> MountingHole_Pad; symbol Mechanical:MountingHole_Pad -> Mechanical:MountingHole
- J5: value (none) -> AUDIO_IN
- U1: value (none) -> TL084; footprint (none) -> Package_DIP:DIP-14_W7.62mm_Socket
Connections:
- net Bias is gone; now on net BIAS: R27.1, U1.14
- net BP: now also R19.1, U2.6 (-), U2.7; no longer R19.2, U2.1, U2.2 (-)
- net GND: now also U2.12 (+); no longer H2.1, U2.10 (+)
- net HP: now also C2.2, U2.8; no longer C2.1, U2.14
- net TP: now also U2.1, U2.3 (+); no longer U2.5 (+), U2.7
- net at RV4.3: now also R14.2; no longer R14.1
- net at C15.1, R16.2, U3.6: now also U2.5 (+); no longer U2.3 (+)
- net at RV3.2: now also C14.2; no longer C14.1
- net at R20.2, R7.1, R9.2: now also U2.9 (-); no longer U2.13 (-)
- net at C16.1, R26.2, U4.6: now also U2.2 (-); no longer U2.6 (-)
- net at U1.9 (-): now also C2.1; no longer C2.2
- net at R1.2: now also R6.2, U2.13 (-); no longer C14.2
- net at R21.2, U4.2 (-): now also R19.2; no longer R19.1
- net at R6.1, R7.2: now also U2.14; no longer U2.8
- new net: R14.1, R8.1, U2.10 (+)
- new net: C14.1, R1.1
Other:
- moved on the sheet: C14, C2, R1, R13, R14, R19

Commit message: Final version 1
Parts:
- added H3: MountingHole_Pad, MountingHole:MountingHole_3.2mm_M3_DIN965, symbol Mechanical:MountingHole
- H2: footprint (none) -> MountingHole:MountingHole_3.2mm_M3_DIN965
- U2: value (none) -> TL084; footprint (none) -> Package_DIP:DIP-14_W7.62mm_Socket
Connections:
- net +12V: now also RV2.3; no longer RV2.1
- net -12V: now also RV2.1; no longer RV2.3
- net AUDIO_IN_ATT: now also RV3.3; no longer RV3.1
- net BP: now also RV4.3; no longer RV4.1
- net FREQ_CV_IN: now also RV1.3; no longer RV1.1
- net GND: now also RV1.1, RV3.1; no longer RV1.3, RV3.3
- net at R14.2: now also RV4.1; no longer RV4.3
Other:
- moved on the sheet: RV4
Changed lines of the file:
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@@
   (junction (at 74.93 173.99) (diameter 0) (color 0 0 0 0)
   )
-  (bus_entry (at 80.01 177.8) (size 2.54 2.54)
-    (stroke (width 0) (type default) (color 0 0 0 0))
-  )
-  (bus_entry (at 87.63 172.72) (size 2.54 2.54)
-    (stroke (width 0) (type default) (color 0 0 0 0))
-  )
   (wire (pts (xy 63.5 48.26) (xy 66.04 48.26))
     (stroke (width 0) (type default) (color 0 0 0 0))
@@
   )
   (wire (pts (xy 77.47 53.34) (xy 73.66 53.34))
-    (stroke (width 0) (type default) (color 0 0 0 0))
-  )
-  (wire (pts (xy 163.83 173.99) (xy 163.83 176.53))
     (stroke (width 0) (type default) (color 0 0 0 0))
   )
@@
     (pin "2")
   )
-  (symbol (lib_id "Device:R_Potentiometer") (at 134.62 73.66 270) (unit 1)
+  (symbol (lib_id "Device:R_Potentiometer") (at 134.62 73.66 90) (mirror x) (unit 1)
     (in_bom yes) (on_board yes) (fields_autoplaced)
     (property "Reference" "RV4" (id 0) (at 134.62 67.31 90))
@@
       (effects (font (size 1.27 1.27)) (justify left))
     )
-    (property "Footprint" "" (id 2) (at 163.83 171.45 0)
+    (property "Footprint" "MountingHole:MountingHole_3.2mm_M3_DIN965" (id 2) (at 163.83 171.45 0)
       (effects (font (size 1.27 1.27)) hide)
     )
@@
     (pin "2")
   )
-  (symbol (lib_id "Device:R_Potentiometer") (at 24.13 45.72 0) (unit 1)
+  (symbol (lib_id "Device:R_Potentiometer") (at 24.13 45.72 0) (mirror x) (unit 1)
     (in_bom yes) (on_board yes) (fields_autoplaced)
     (property "Reference" "RV3" (id 0) (at 21.59 44.4499 0)
@@
     (in_bom yes) (on_board yes) (fields_autoplaced)
     (property "Reference" "U2" (id 0) (at 85.09 40.64 0))
-    (property "Value" "" (id 1) (at 85.09 43.18 0))
-    (property "Footprint" "" (id 2) (at 83.82 53.34 0)
+    (property "Value" "TL084" (id 1) (at 85.09 43.18 0))
+    (property "Footprint" "Package_DIP:DIP-14_W7.62mm_Socket" (id 2) (at 83.82 53.34 0)
       (effects (font (size 1.27 1.27)) hide)
     )
@@
     (pin "1")
   )
-  (symbol (lib_id "power:GND") (at 163.83 176.53 0) (unit 1)
-    (in_bom yes) (on_board yes) (fields_autoplaced)
-    (property "Reference" "#PWR0103" (id 0) (at 163.83 182.88 0)
-      (effects (font (size 1.27 1.27)) hide)
-    )
-    (property "Value" "GND" (id 1) (at 163.83 181.61 0))
-    (property "Footprint" "" (id 2) (at 163.83 176.53 0)
-      (effects (font (size 1.27 1.27)) hide)
-    )
-    (property "Datasheet" "" (id 3) (at 163.83 176.53 0)
-      (effects (font (size 1.27 1.27)) hide)
-    )
-    (pin "1")
-  )
   (symbol (lib_id "Device:R_Small") (at 220.98 57.15 180) (unit 1)
     (in_bom yes) (on_board yes)
@@
     (in_bom yes) (on_board yes) (fields_autoplaced)
     (property "Reference" "U2" (id 0) (at 161.29 40.64 0))
-    (property "Value" "" (id 1) (at 161.29 43.18 0))
-    (property "Footprint" "" (id 2) (at 160.02 53.34 0)
+    (property "Value" "TL084" (id 1) (at 161.29 43.18 0))
+    (property "Footprint" "Package_DIP:DIP-14_W7.62mm_Socket" (id 2) (at 160.02 53.34 0)
       (effects (font (size 1.27 1.27)) hide)
     )
@@
       (effects (font (size 1.27 1.27)) (justify left))
     )
-    (property "Value" "" (id 1) (at 31.75 176.5299 0)
-      (effects (font (size 1.27 1.27)) (justify left))
-    )
-    (property "Footprint" "" (id 2) (at 31.75 172.72 0)
+    (property "Value" "TL084" (id 1) (at 31.75 176.5299 0)
+      (effects (font (size 1.27 1.27)) (justify left))
+    )
+    (property "Footprint" "Package_DIP:DIP-14_W7.62mm_Socket" (id 2) (at 31.75 172.72 0)
       (effects (font (size 1.27 1.27)) hide)
     )
@@
     (pin "1")
   )
+  (symbol (lib_id "Mechanical:MountingHole") (at 163.83 177.8 0) (unit 1)
+    (in_bom yes) (on_board yes) (fields_autoplaced)
+    (property "Reference" "H3" (id 0) (at 166.37 176.5299 0)
+      (effects (font (size 1.27 1.27)) (justify left))
+    )
+    (property "Value" "MountingHole_Pad" (id 1) (at 166.37 179.0699 0)
+      (effects (font (size 1.27 1.27)) (justify left))
+    )
+    (property "Footprint" "MountingHole:MountingHole_3.2mm_M3_DIN965" (id 2) (at 163.83 177.8 0)
+      (effects (font (size 1.27 1.27)) hide)
+    )
+    (property "Datasheet" "~" (id 3) (at 163.83 177.8 0)
+      (effects (font (size 1.27 1.27)) hide)
+    )
+  )
   (symbol (lib_id "Amplifier_Operational:TL084") (at 236.22 50.8 0) (unit 1)
     (in_bom yes) (on_board yes) (fields_autoplaced)
     (property "Reference" "U2" (id 0) (at 236.22 40.64 0))
-    (property "Value" "" (id 1) (at 236.22 43.18 0))
-    (property "Footprint" "" (id 2) (at 234.95 48.26 0)
+    (property "Value" "TL084" (id 1) (at 236.22 43.18 0))
+    (property "Footprint" "Package_DIP:DIP-14_W7.62mm_Socket" (id 2) (at 234.95 48.26 0)
       (effects (font (size 1.27 1.27)) hide)
     )
@@
     (pin "4")
   )
-  (symbol (lib_id "Device:R_Potentiometer") (at 181.61 147.32 0) (unit 1)
+  (symbol (lib_id "Device:R_Potentiometer") (at 181.61 147.32 0) (mirror x) (unit 1)
     (in_bom yes) (on_board yes) (fields_autoplaced)
     (property "Reference" "RV1" (id 0) (at 179.07 146.0499 0)
@@
     (pin "2")
   )
-  (symbol (lib_id "Device:R_Potentiometer") (at 193.04 133.35 0) (unit 1)
+  (symbol (lib_id "Device:R_Potentiometer") (at 193.04 133.35 0) (mirror x) (unit 1)
     (in_bom yes) (on_board yes) (fields_autoplaced)
     (property "Reference" "RV2" (id 0) (at 190.5 132.0799 0)
@@
     (in_bom yes) (on_board yes) (fields_autoplaced)
     (property "Reference" "U2" (id 0) (at 55.88 38.1 0))
-    (property "Value" "" (id 1) (at 55.88 40.64 0))
-    (property "Footprint" "" (id 2) (at 54.61 50.8 0)
+    (property "Value" "TL084" (id 1) (at 55.88 40.64 0))
+    (property "Footprint" "Package_DIP:DIP-14_W7.62mm_Socket" (id 2) (at 54.61 50.8 0)
       (effects (font (size 1.27 1.27)) hide)
     )
@@
       (reference "#PWR0102") (unit 1) (value "+12V") (footprint "")
     )
-    (path "/4f9772d0-1425-4549-a153-d031195742f5"
-      (reference "#PWR0103") (unit 1) (value "GND") (footprint "")
-    )
     (path "/5d9fdbd7-23f7-4aa0-94d9-419292e84138"
       (reference "#PWR0104") (unit 1) (value "GND") (footprint "")
@@
       (reference "H2") (unit 1) (value "MountingHole_Pad") (footprint "MountingHole:MountingHole_3.2mm_M3_DIN965")
     )
+    (path "/812aca2d-68c2-4d32-aeb1-34311912c908"
+      (reference "H3") (unit 1) (value "MountingHole_Pad") (footprint "MountingHole:MountingHole_3.2mm_M3_DIN965")
+    )
     (path "/d03a111d-fcbc-4bca-b811-e5a1cdd30de8"

Commit message: Final v2
Connections:
- net GND: now also H1.3, H1.4, H1.5, H1.6, H1.7, H1.8
- net TP: now also U2.2 (-); no longer U2.3 (+)
- net at C16.1, R26.2, U4.6: now also U2.3 (+); no longer U2.2 (-)
- net at R4.2, R5.1: now also U1.9 (-); no longer U1.10 (+)
- net at C2.1: now also U1.10 (+); no longer U1.9 (-)
Other:
- moved on the sheet: H2, H3
Changed lines of the file:
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@@
+    (stroke (width 0) (type default) (color 0 0 0 0))
+  )
+  (wire (pts (xy 137.16 171.45) (xy 132.08 171.45))
     (stroke (width 0) (type default) (color 0 0 0 0))
   )
@@
   )
   (wire (pts (xy 114.3 168.91) (xy 132.08 168.91))
+    (stroke (width 0) (type default) (color 0 0 0 0))
+  )
+  (wire (pts (xy 137.16 172.72) (xy 137.16 171.45))
     (stroke (width 0) (type default) (color 0 0 0 0))
   )
@@
     (pin "1")
   )
-  (symbol (lib_id "Mechanical:MountingHole") (at 163.83 171.45 0) (unit 1)
-    (in_bom yes) (on_board yes) (fields_autoplaced)
-    (property "Reference" "H2" (id 0) (at 166.37 170.1799 0)
-      (effects (font (size 1.27 1.27)) (justify left))
-    )
-    (property "Value" "MountingHole_Pad" (id 1) (at 166.37 172.7199 0)
-      (effects (font (size 1.27 1.27)) (justify left))
-    )
-    (property "Footprint" "MountingHole:MountingHole_3.2mm_M3_DIN965" (id 2) (at 163.83 171.45 0)
-      (effects (font (size 1.27 1.27)) hide)
-    )
-    (property "Datasheet" "~" (id 3) (at 163.83 171.45 0)
+  (symbol (lib_id "Mechanical:MountingHole") (at 151.13 170.18 0) (unit 1)
+    (in_bom yes) (on_board yes) (fields_autoplaced)
+    (property "Reference" "H2" (id 0) (at 153.67 168.9099 0)
+      (effects (font (size 1.27 1.27)) (justify left))
+    )
+    (property "Value" "MountingHole_Pad" (id 1) (at 153.67 171.4499 0)
+      (effects (font (size 1.27 1.27)) (justify left))
+    )
+    (property "Footprint" "MountingHole:MountingHole_3.2mm_M3_DIN965" (id 2) (at 151.13 170.18 0)
+      (effects (font (size 1.27 1.27)) hide)
+    )
+    (property "Datasheet" "~" (id 3) (at 151.13 170.18 0)
       (effects (font (size 1.27 1.27)) hide)
     )
@@
     (pin "4")
   )
-  (symbol (lib_id "Amplifier_Operational:TL084") (at 33.02 135.89 0) (mirror x) (unit 3)
+  (symbol (lib_id "Amplifier_Operational:TL084") (at 33.02 135.89 0) (unit 3)
     (in_bom yes) (on_board yes) (fields_autoplaced)
     (property "Reference" "U1" (id 0) (at 33.02 125.73 0))
     (property "Value" "TL084" (id 1) (at 33.02 128.27 0))
-    (property "Footprint" "Package_DIP:DIP-14_W7.62mm_Socket" (id 2) (at 31.75 138.43 0)
-      (effects (font (size 1.27 1.27)) hide)
-    )
-    (property "Datasheet" "http://www.ti.com/lit/ds/symlink/tl081.pdf" (id 3) (at 34.29 140.97 0)
+    (property "Footprint" "Package_DIP:DIP-14_W7.62mm_Socket" (id 2) (at 31.75 133.35 0)
+      (effects (font (size 1.27 1.27)) hide)
+    )
+    (property "Datasheet" "http://www.ti.com/lit/ds/symlink/tl081.pdf" (id 3) (at 34.29 130.81 0)
       (effects (font (size 1.27 1.27)) hide)
     )
@@
     (pin "1")
   )
-  (symbol (lib_id "Mechanical:MountingHole") (at 163.83 177.8 0) (unit 1)
-    (in_bom yes) (on_board yes) (fields_autoplaced)
-    (property "Reference" "H3" (id 0) (at 166.37 176.5299 0)
-      (effects (font (size 1.27 1.27)) (justify left))
-    )
-    (property "Value" "MountingHole_Pad" (id 1) (at 166.37 179.0699 0)
-      (effects (font (size 1.27 1.27)) (justify left))
-    )
-    (property "Footprint" "MountingHole:MountingHole_3.2mm_M3_DIN965" (id 2) (at 163.83 177.8 0)
-      (effects (font (size 1.27 1.27)) hide)
-    )
-    (property "Datasheet" "~" (id 3) (at 163.83 177.8 0)
-      (effects (font (size 1.27 1.27)) hide)
-    )
-  )
-  (symbol (lib_id "Amplifier_Operational:TL084") (at 236.22 50.8 0) (unit 1)
+  (symbol (lib_id "Mechanical:MountingHole") (at 151.13 176.53 0) (unit 1)
+    (in_bom yes) (on_board yes) (fields_autoplaced)
+    (property "Reference" "H3" (id 0) (at 153.67 175.2599 0)
+      (effects (font (size 1.27 1.27)) (justify left))
+    )
+    (property "Value" "MountingHole_Pad" (id 1) (at 153.67 177.7999 0)
+      (effects (font (size 1.27 1.27)) (justify left))
+    )
+    (property "Footprint" "MountingHole:MountingHole_3.2mm_M3_DIN965" (id 2) (at 151.13 176.53 0)
+      (effects (font (size 1.27 1.27)) hide)
+    )
+    (property "Datasheet" "~" (id 3) (at 151.13 176.53 0)
+      (effects (font (size 1.27 1.27)) hide)
+    )
+  )
+  (symbol (lib_id "Amplifier_Operational:TL084") (at 236.22 50.8 0) (mirror x) (unit 1)
     (in_bom yes) (on_board yes) (fields_autoplaced)
     (property "Reference" "U2" (id 0) (at 236.22 40.64 0))
     (property "Value" "TL084" (id 1) (at 236.22 43.18 0))
-    (property "Footprint" "Package_DIP:DIP-14_W7.62mm_Socket" (id 2) (at 234.95 48.26 0)
-      (effects (font (size 1.27 1.27)) hide)
-    )
-    (property "Datasheet" "http://www.ti.com/lit/ds/symlink/tl081.pdf" (id 3) (at 237.49 45.72 0)
+    (property "Footprint" "Package_DIP:DIP-14_W7.62mm_Socket" (id 2) (at 234.95 53.34 0)
+      (effects (font (size 1.27 1.27)) hide)
+    )
+    (property "Datasheet" "http://www.ti.com/lit/ds/symlink/tl081.pdf" (id 3) (at 237.49 55.88 0)
       (effects (font (size 1.27 1.27)) hide)
     )
@@
     (pin "1")
   )
+  (symbol (lib_id "power:GND") (at 137.16 172.72 0) (unit 1)
+    (in_bom yes) (on_board yes) (fields_autoplaced)
+    (property "Reference" "#PWR?" (id 0) (at 137.16 179.07 0)
+      (effects (font (size 1.27 1.27)) hide)
+    )
+    (property "Value" "GND" (id 1) (at 137.16 177.8 0))
+    (property "Footprint" "" (id 2) (at 137.16 172.72 0)
+      (effects (font (size 1.27 1.27)) hide)
+    )
+    (property "Datasheet" "" (id 3) (at 137.16 172.72 0)
+      (effects (font (size 1.27 1.27)) hide)
+    )
+    (pin "1")
+  )
   (symbol (lib_id "power:GND") (at 43.18 151.13 0) (unit 1)
     (in_bom yes) (on_board yes) (fields_autoplaced)
@@
       (reference "#PWR0105") (unit 1) (value "GND") (footprint "")
     )
+    (path "/d6b39609-7178-48e0-aa23-b170b31b5b76"
+      (reference "#PWR?") (unit 1) (value "GND") (footprint "")
+    )
     (path "/c5b0f823-2c30-42d4-b7d2-e1f9af885781"
