File: VCF.kicad_pcb (KiCad board)
At the start: 2 copper layers, 58 x 105 mm, 57 parts, among them J1 CV_IN, J2 TP_OUT, J3 BP_OUT, J4 HP_OUT, J5 AUDIO_IN, U1 TL084, U2 TL084, U3 CA3080, U4 CA3080

Commit message: Final version 1
Parts:
- added H3: MountingHole_Pad, MountingHole:MountingHole_3.2mm_M3_DIN965, F.Cu at (102.0, 52.8)
- C11, C9: moved to B.Cu
- moved C5 15.3 mm to (63.5, 55.9), turned to 90 degrees
- moved C16 9.78 mm to (92.8, 108.2)
- moved C12 9.48 mm to (81.3, 53.4), turned to -90 degrees
- moved C9 8.78 mm to (77.5, 58.4), turned to 90 degrees
- moved R16 7.24 mm to (102.9, 101.3)
- moved C15 6.86 mm to (93.0, 98.0)
- moved H1 6.47 mm to (96.5, 54.6)
- moved R26 3.18 mm to (102.9, 104.8)
- moved C4 1.50 mm to (71.1, 53.3)
Connections:
- RV1 pad 1: /FREQ_CV_IN -> GND
- RV1 pad 3: GND -> /FREQ_CV_IN
- RV2 pad 1: +12V -> -12V
- RV2 pad 3: -12V -> +12V
- RV3 pad 1: /AUDIO_IN_ATT -> GND
- RV3 pad 3: GND -> /AUDIO_IN_ATT
- RV4 pad 1: /BP -> Net-(R14-Pad2)
- RV4 pad 3: Net-(R14-Pad2) -> /BP
Routing:
- net +12V: track 186.9 -> 169.2 mm
- net Net-(C16-Pad1): track 43.1 -> 49.6 mm
- net GND: track 6.44 -> 0.00 mm
- net Net-(R14-Pad2): track 35.2 -> 30.2 mm
- net /BP: track 145.0 -> 147.7 mm
- net -12V: track 142.9 -> 145.0 mm
- net Net-(C15-Pad1): track 21.9 -> 20.2 mm
- net /TP: track 56.1 -> 57.6 mm
- net Net-(R22-Pad1): track 70.4 -> 69.3 mm
